File: Water Quality Measurement/Water Quality Measurement.kicad_pcb (KiCad board)
At the start: 2 copper layers, 99.8 x 72.1 mm, 17 parts, among them J1 pH Sensor, J2 OLED Screen, J3 MountingPin_IO1, J4 Conn_01x02_MountingPin, J5 MountingPin_IO46, J6 9V Battery Enclosure, J7 Conn_01x02_MountingPin, J8 9V Battery Enclosure, Q1 PMV15UNEAR, U1 LM7805_TO220

Commit message: Add files via upload
Parts:
- removed J3: MountingPin_IO1, Connector_PinHeader_2.54mm:PinHeader_1x20_P2.54mm_Vertical
- removed J5: MountingPin_IO46, Connector_PinHeader_2.54mm:PinHeader_1x20_P2.54mm_Vertical
- removed J8: 9V Battery Enclosure, Connector_PinHeader_2.54mm:PinHeader_1x02_P2.54mm_Vertical
- added J10: 9V Enclosure, Connector_PinHeader_2.54mm:PinHeader_1x02_P2.54mm_Vertical, F.Cu at (127.3, 50.3)
- added J11: Water Pump - OUT, Connector_PinHeader_2.54mm:PinHeader_1x02_P2.54mm_Vertical, F.Cu at (107.7, 50.8)
- added J12: 9V Enclosure, Connector_PinHeader_2.54mm:PinHeader_1x02_P2.54mm_Vertical, F.Cu at (119.4, 54.6)
- added R2: 4.7k, Resistor_SMD:R_2010_5025Metric, F.Cu at (133.6, 91.9)
- added R3: 4.7k, Resistor_SMD:R_2010_5025Metric, F.Cu at (152.4, 76.2)
- J1: value pH Sensor -> OLED Screen; footprint Connector_PinHeader_2.54mm:PinHeader_1x03_P2.54mm_Vertical -> Connector_PinHeader_2.54mm:PinHeader_1x04_P2.54mm_Vertical
- J2: value OLED Screen -> DevBoard Left; footprint Connector_PinHeader_2.54mm:PinHeader_1x04_P2.54mm_Vertical -> Connector_PinHeader_2.54mm:PinHeader_1x20_P2.54mm_Vertical
- J4: value Conn_01x02_MountingPin -> Water Pump - IN
- J6: value 9V Battery Enclosure -> pH Sensor; footprint Connector_PinHeader_2.54mm:PinHeader_1x02_P2.54mm_Vertical -> Connector_PinHeader_2.54mm:PinHeader_1x03_P2.54mm_Vertical
- J7: value Conn_01x02_MountingPin -> DevBoard Right; footprint Connector_PinHeader_2.54mm:PinHeader_1x02_P2.54mm_Vertical -> Connector_PinHeader_2.54mm:PinHeader_1x20_P2.54mm_Vertical
- R1: value 1k -> 100; footprint Resistor_SMD:R_2512_6332Metric -> Resistor_SMD:R_1206_3216Metric
- U1: value LM7805_TO220 -> Voltage regulator
- moved J6 64.4 mm to (177.5, 112.0), turned to -90 degrees
- moved C1 60.6 mm to (126.0, 57.9)
- moved C2 43.7 mm to (150.4, 65.8), turned to 0 degrees
- moved J1 43.5 mm to (142.8, 84.8), turned to 90 degrees
- moved J4 43.5 mm to (95.2, 50.8)
- moved R1 40.6 mm to (103.1, 115.6)
- moved Q1 40.5 mm to (114.1, 114.3)
- moved U1 16.4 mm to (142.2, 60.5)
- moved J2 14.6 mm to (96.5, 62.2), turned to 0 degrees
- moved J7 10.6 mm to (127.0, 62.2)
Connections:
- C1 pad 1: Net-(J8-Pin_1) -> /5V
- C2 pad 1: Net-(J4-Pin_1) -> Net-(J10-Pin_1)
- J1 pad 1: GND -> /3.3
- J1 pad 2: /3.3 -> GND
- J1 pad 3: pH sen. input -> SCL
- J2 pad 1: /3.3 -> unconnected-(J2-Pin_1-Pad1)
- J2 pad 2: GND -> unconnected-(J2-Pin_2-Pad2)
- J2 pad 3: SCL -> unconnected-(J2-Pin_3-Pad3)
- J2 pad 4: SDA -> unconnected-(J2-Pin_4-Pad4)
- J4 pad 1: Net-(J4-Pin_1) -> Net-(J10-Pin_1)
- J4 pad 2: Net-(J4-Pin_2) -> Net-(J11-Pin_2)
- J6 pad 1: Net-(J4-Pin_1) -> GND
- J6 pad 2: GND -> /3.3
- J7 pad 1: Net-(J4-Pin_1) -> unconnected-(J7-Pin_1-Pad1)
- J7 pad 2: Net-(J4-Pin_2) -> unconnected-(J7-Pin_2-Pad2)
- Q1 pad 3: Net-(J4-Pin_2) -> Net-(J11-Pin_2)
- U1 pad 1: Net-(J4-Pin_1) -> Net-(J10-Pin_1)
- U1 pad 3: Net-(J8-Pin_1) -> /5V
Routing:
- net GND: track 243.4 -> 5.18 mm, vias 2 -> 3
- net /3.3: track 139.6 -> 0.00 mm
- net Net-(J4-Pin_1): track 108.0 -> 0.00 mm
- net Net-(J11-Pin_2): track 0.00 -> 98.7 mm
- net Net-(J10-Pin_1): track 0.00 -> 62.2 mm
- net Net-(J8-Pin_1): track 43.5 -> 0.00 mm
- net Net-(J4-Pin_2): track 42.8 -> 0.00 mm
- net pH sen. input: track 88.5 -> 57.6 mm
- net Net-(Q1-G): track 27.3 -> 9.52 mm
- net SDA: track 29.5 -> 36.5 mm
- net /IO26: track 12.1 -> 18.9 mm
- added copper zone on F.Cu, net /3.3
- added copper zone on F.Cu, net /5V
