File: Water Quality Measurement/Water Quality Measurement.kicad_sch (KiCad schematic)
At the start: 17 parts, among them J1 pH Sensor, J2 OLED Screen, J3 MountingPin_IO1, J4 Conn_01x02_MountingPin, J5 MountingPin_IO46, J6 9V Battery Enclosure, J7 Conn_01x02_MountingPin, J8 9V Battery Enclosure, Q1 PMV15UNEAR, U1 LM7805_TO220

Commit message: Add files via upload
Parts:
- removed J1: pH Sensor, Connector_PinHeader_2.54mm:PinHeader_1x03_P2.54mm_Vertical, symbol Connector_Generic_MountingPin:Conn_01x03_MountingPin
- removed J2: OLED Screen, Connector_PinHeader_2.54mm:PinHeader_1x04_P2.54mm_Vertical, symbol Connector_Generic_MountingPin:Conn_01x04_MountingPin
- removed J3: MountingPin_IO1, Connector_PinHeader_2.54mm:PinHeader_1x20_P2.54mm_Vertical, symbol Connector_Generic_MountingPin:Conn_01x20_MountingPin
- removed J4, J7: Conn_01x02_MountingPin, Connector_PinHeader_2.54mm:PinHeader_1x02_P2.54mm_Vertical, symbol Connector_Generic_MountingPin:Conn_01x02_MountingPin
- removed J5: MountingPin_IO46, Connector_PinHeader_2.54mm:PinHeader_1x20_P2.54mm_Vertical, symbol Connector_Generic_MountingPin:Conn_01x20_MountingPin
- removed J6, J8: 9V Battery Enclosure, Connector_PinHeader_2.54mm:PinHeader_1x02_P2.54mm_Vertical, symbol Connector_Generic_MountingPin:Conn_01x02_MountingPin
- added J1: OLED Screen, Connector_PinHeader_2.54mm:PinHeader_1x04_P2.54mm_Vertical, symbol Connector_Generic:Conn_01x04
- added J10, J12: 9V Enclosure, Connector_PinHeader_2.54mm:PinHeader_1x02_P2.54mm_Vertical, symbol Connector_Generic:Conn_01x02
- added J11: Water Pump - OUT, Connector_PinHeader_2.54mm:PinHeader_1x02_P2.54mm_Vertical, symbol Connector_Generic:Conn_01x02
- added J2: DevBoard Left, Connector_PinHeader_2.54mm:PinHeader_1x20_P2.54mm_Vertical, symbol Connector_Generic:Conn_01x20
- added J4: Water Pump - IN, Connector_PinHeader_2.54mm:PinHeader_1x02_P2.54mm_Vertical, symbol Connector_Generic:Conn_01x02
- added J6: pH Sensor, Connector_PinHeader_2.54mm:PinHeader_1x03_P2.54mm_Vertical, symbol Connector_Generic:Conn_01x03
- added J7: DevBoard Right, Connector_PinHeader_2.54mm:PinHeader_1x20_P2.54mm_Vertical, symbol Connector_Generic:Conn_01x20
- added R2, R3: 4.7k, Resistor_SMD:R_2010_5025Metric, symbol Device:R_US
- R1: value 1k -> 100; footprint Resistor_SMD:R_2512_6332Metric -> Resistor_SMD:R_1206_3216Metric
- U1: value LM7805_TO220 -> Voltage regulator
Connections:
- net 3.3: now also J1.1 (Pin_1), J6.2 (Pin_2), J7.19 (Pin_19), R2.2, R3.2
- net GND: now also J1.2 (Pin_2), J10.2 (Pin_2), J12.2 (Pin_2), J2.20 (Pin_20), J6.1 (Pin_1), J7.20 (Pin_20)
- net IO26: now also J2.17 (Pin_17)
- net SCL: now also J1.3 (Pin_3), J7.9 (Pin_9), R2.1
- net SDA: now also J1.4 (Pin_4), J7.8 (Pin_8), R3.1
- net pH sen. input: now also J6.3 (Pin_3), J7.17 (Pin_17)
- net at C2.1, U1.1 (VI): now also J10.1 (Pin_1), J11.1 (Pin_1), J4.1 (Pin_1)
- net at Q1.3 (D): now also J11.2 (Pin_2), J4.2 (Pin_2)
- net 5V: now reaches C1.1, U1.3 (VO)
- net 5V: now also J12.1 (Pin_1), J2.19 (Pin_19)
- no-connect marks 0 -> 32
